Commit message: create the birl_baxter_common   by ben

File: birl_baxter_description/urdf/ft/robots/FT_Electric_left.URDF (robot description, URDF)
Before this commit: robot FT_Electric_left, 3 links, 2 joints
Joints:
- joint FT_Top_Joint_left: axis (none) -> 0 0 1; limit (none) -> lower=0 upper=0.0006 effort=0.001 velocity=0.001; type fixed -> prismatic

File: birl_baxter_description/urdf/ft/robots/FT_Electric_right.URDF (robot description, URDF)
Before this commit: robot FT_Electric_right, 3 links, 2 joints
Joints:
- joint FT_Top_Joint_right: axis (none) -> 0 0 1; limit (none) -> lower=0 upper=0.0006 effort=0.001 velocity=0.001
