Commit message: fixed box frame, finish all launch files

File: birl_baxter_description/urdf/box/box_female/robots/box_female.URDF (robot description, URDF)
Before this commit: robot box_female, 1 links, 1 joints
Links:
- removed link left_box_female
- added link box_female, mass 0.01501; collision mesh filename=package://birl_baxter_description/urdf/box/box_female/meshe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; visual mesh filename=package://birl_baxter_description/urdf/box/box_female/meshe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
Joints:
- removed joint left_female_box_joint
- added joint female_box_joint: type fixed, parent base, child box_female, origin xyz=0.6 0 -0.115 rpy=0 0 0

File: birl_baxter_description/urdf/box/box_male/robots/box_male.URDF (robot description, URDF)
Before this commit: robot box_male, 1 links, 1 joints
Links:
- removed link box_male
- added link left_box_male, mass 0.01526; collision mesh filename=package://birl_baxter_description/urdf/box/box_male/meshes/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; visual mesh filename=package://birl_baxter_description/urdf/box/box_male/meshes/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
Joints:
- removed joint male_box_joint
- added joint left_male_box_joint: type fixed, parent left_female_holder, child left_box_male, origin xyz=0 0 0.015 rpy=0 0 0
