Commit message: pick and place box demo launch

File: birl_baxter_description/urdf/asus_xtion/asus_xtion.xacro (robot description, xacro)
@@ -59,9 +59,9 @@
     </inertial>
   </link>
-  <joint name="camera_base_fixed" type="fixed">
+<!--  <joint name="camera_base_fixed" type="fixed">
     <origin rpy="0 0 0" xyz="1.0 0.0 -0.93"/>
     <parent link="base"/>
     <child link="camera_base"/>
-  </joint>
+  </joint>-->
   <joint name="install_link_fixed" type="fixed">
     <origin rpy="0 0 0" xyz="-0.35 -0.05 1.5"/>

File: birl_baxter_description/urdf/baxter_element/baxter_base/baxter_base_ft.urdf.xacro (robot description, xacro)
@@ -1006,6 +1006,6 @@
     <gazebo>
       <plugin name="ft_sensor_right" filename="libgazebo_ros_ft_sensor.so">
-        <updateRate>10.0</updateRate>
-        <topicName>ft_sensor_topic_right</topicName>
+        <updateRate>200.0</updateRate>
+        <topicName>wrench/filtered/right</topicName>
         <jointName>right_w2</jointName>
       </plugin>
@@ -1034,12 +1034,12 @@
       <child link="FT_bottom_plate_left"/>
     </joint>
-    <gazebo reference="FT_Top_Joint_left">
+    <gazebo reference="left_w2">
       <provideFeedback>true</provideFeedback>
     </gazebo>
     <gazebo>
       <plugin name="ft_sensor_left" filename="libgazebo_ros_ft_sensor.so">
-        <updateRate>10.0</updateRate>
-        <topicName>ft_sensor_topic_left</topicName>
-        <jointName>FT_Top_Joint_left</jointName>
+        <updateRate>200.0</updateRate>
+        <topicName>wrench/filtered/left</topicName>
+        <jointName>left_w2</jointName>
       </plugin>
     </gazebo>

File: birl_baxter_description/urdf/baxter_element/baxter_pa/baxter_pa_box2.urdf.xacro (robot description, xacro)
@@ -8,9 +8,9 @@
   <xacro:arg name="right_camera_frame" default="true"/>
   <xacro:arg name="left_camera_frame" default="true"/>
-  <xacro:arg name="left_male_holder" default="true"/>
-  <xacro:arg name="right_male_holder" default="true"/>
-  <xacro:arg name="l_finger"       default="pa_finger"/>
-  <xacro:arg name="l_finger_slot"  default="6"/>
-  <xacro:arg name="l_finger_tip"   default="pa_tip"/>
+  <xacro:arg name="left_male_holder" default="false"/>
+  <xacro:arg name="right_male_holder" default="false"/>
+  <xacro:arg name="l_finger"       default="standard_narrow"/>
+  <xacro:arg name="l_finger_slot"  default="4"/>
+  <xacro:arg name="l_finger_tip"   default="paddle_tip"/>
   <xacro:arg name="l_finger_grasp" default="inner"/>
   <xacro:arg name="r_finger"       default="pa_finger"/>
@@ -18,5 +18,9 @@
   <xacro:arg name="r_finger_tip"   default="pa_tip"/>
   <xacro:arg name="r_finger_grasp" default="inner"/>
-  <xacro:arg name="left_ft_sensor" default="false"/>
+  <!--options:
+      finger = extended_wide extended_narrow standard_narrow standard_wide pa_finger
+      finger_slot = 1-6
+      fing_tip = basic_hard_tip basic_soft_tip half_round_tip paddle_tip none-->
+  <xacro:arg name="left_ft_sensor" default="true"/>
   <xacro:arg name="right_ft_sensor" default="true"/>
   <!-- Baxter Base URDF -->
@@ -50,12 +54,4 @@
       <xacro:arg name="r_finger_grasp" default="$(r_finger_grasp)"/>
     </xacro:include>
-    <xacro:include filename="$(find birl_baxter_description)/urdf/box/box_male/robots/box_male.URDF" >
-    </xacro:include>
-  <joint name="left_male_box_joint" type="fixed">
-      <origin rpy="0 0 0" xyz="0 0 0.015"/>
-      <parent link="left_male_holder" />
-      <child link="left_box_male"/>
-  </joint>
-  <!-- Table -->
   <xacro:if value="$(arg table)">
     <xacro:include filename="$(find birl_baxter_description)/urdf/table/table.xacro">
@@ -77,10 +73,3 @@
     </joint>
   </xacro:if>
-      <xacro:include filename="$(find birl_baxter_description)/urdf/box/box_female/robots/box_female.URDF" >
-    </xacro:include>
-    <joint name="female_box_joint" type="fixed">
-      <origin rpy="0 0 0" xyz="0.6 0 -0.115"/>
-      <parent link="base" />
-      <child link="box_female"/>
-    </joint>
 </robot>

File: birl_baxter_description/urdf/baxter_element/left_end_pa_effector.urdf.xacro (robot description, xacro)
@@ -6,4 +6,5 @@
   <xacro:arg name="l_finger_grasp" default="inner"/>
   <xacro:arg name="left_camera_frame" default="false"/>
+  <xacro:arg name="left_male_holder" default="false"/>
   <xacro:include filename="$(find birl_gripper_description)/urdf/electric_gripper/rethink_electric_pa_gripper.xacro" />
   <xacro:rethink_electric_gripper side="left"
@@ -16,4 +17,5 @@
                                   r_finger_tip="$(arg l_finger_tip)"
                                   r_finger_grasp="$(arg l_finger_grasp)"
-                                  camera_frame="$(arg left_camera_frame)"/>
+                                  camera_frame="$(arg left_camera_frame)"
+                                  male_holder="$(arg left_male_holder)" />
 </robot>

File: birl_baxter_description/urdf/baxter_element/right_end_pa_effector.urdf.xacro (robot description, xacro)
@@ -6,4 +6,5 @@
   <xacro:arg name="r_finger_grasp" default="inner"/>
   <xacro:arg name="right_camera_frame" default="false"/>
+  <xacro:arg name="right_male_holder" default="false"/>
   <xacro:include filename="$(find birl_gripper_description)/urdf/electric_gripper/rethink_electric_pa_gripper.xacro" />
   <xacro:rethink_electric_gripper side="right"
@@ -16,4 +17,5 @@
                                   r_finger_tip="$(arg r_finger_tip)"
                                   r_finger_grasp="$(arg r_finger_grasp)"
-                                  camera_frame="$(arg right_camera_frame)"/>
+                                  camera_frame="$(arg right_camera_frame)"
+                                  male_holder="$(arg right_male_holder)"/>
 </robot>

File: birl_baxter_description/urdf/box/box_female/robots/box_female.URDF (robot description, URDF)
Before this commit: robot box_female, 1 links, 1 joints
Joints:
- removed joint female_box_joint

File: birl_baxter_description/urdf/box/box_male/robots/box_male.URDF (robot description, URDF)
Before this commit: robot left_box_male, 1 links, 1 joints
Joints:
- removed joint left_male_box_joint

File: birl_baxter_description/urdf/ft/robots/FT_Electric_left.URDF (robot description, URDF)
Before this commit: robot FT_Electric_left, 3 links, 2 joints
Joints:
- joint FT_Top_Joint_left: type prismatic -> fixed

File: birl_baxter_description/urdf/table/table.xacro (robot description, xacro)
@@ -20,12 +20,16 @@
     </inertial>
   </link>
-  <joint name="table_fixed" type="fixed">
+ <!-- <joint name="table_fixed" type="fixed">
     <origin rpy="0 0 0" xyz="0.0 0.0 -0.93"/>
     <parent link="base"/>
     <child link="table"/>
-  </joint>
-<!--    <gazebo reference="table">
-    <selfCollide>true</selfCollide>
+  </joint>-->
+  <gazebo reference="table">
+    <self_collide>1</self_collide>
+    <mu1>1000000</mu1>
+    <mu2>1000000</mu2>
+    <fdir1>0.0 0.0 1.0</fdir1>
+    <kp>1e5</kp>
+    <kd>1.0</kd>
   </gazebo>
-  -->
 </robot>

File: birl_gripper_description/urdf/electric_gripper/fingers/pa_finger.xacro (robot description, xacro)
@@ -27,6 +27,5 @@
       <mu2>1000</mu2>
       <fdir1>0.0 0.0 1.0</fdir1>
-      <kp>1e5</kp>
-      <kd>1.0</kd>
+      <self_collide>1</self_collide>
     </gazebo>
    <xacro:property name="none" value="[none, false, null, empty]" scope="local"/>

File: birl_gripper_description/urdf/electric_gripper/fingers/pa_tip.xacro (robot description, xacro)
@@ -25,4 +25,7 @@
       </inertial>
     </link>
+    <gazebo reference="${parent_link}_tip">
+      <material>Gazebo/Red</material>
+    </gazebo>
     <joint name="${parent_link}_tip_joint" type="fixed">
       <xacro:insert_block name="joint_origin" />

File: birl_gripper_description/urdf/electric_gripper/rethink_electric_pa_gripper.xacro (robot description, xacro)
@@ -1,5 +1,5 @@
 <?xml version="1.0"?>
 <robot xmlns:xacro="http://www.ros.org/wiki/xacro" name="rethink_electric_gripper">
-  <xacro:macro name="rethink_electric_gripper" params="side r_finger r_finger_slot r_finger_tip r_finger_grasp l_finger l_finger_slot l_finger_tip l_finger_grasp camera_frame">
+  <xacro:macro name="rethink_electric_gripper" params="side r_finger r_finger_slot r_finger_tip r_finger_grasp l_finger l_finger_slot l_finger_tip l_finger_grasp camera_frame male_holder">
     <xacro:property name="gripper_side" value="${side[0]}" scope="local"/>
     <!-- Base of end effector -->
@@ -27,5 +27,4 @@
     </link>
         <!--camera frame  -->
-    <xacro:if value="${camera_frame}">
 <!--        <link name="${side}_gripper_base1">
           <visual>
@@ -56,102 +55,137 @@
     </joint>
 -->
+<xacro:if value="${camera_frame}">
   <link name="${side}_camera_frame">
     <inertial>
       <origin
-        xyz="0.024842 -0.00021599 0.048722"
-        rpy="0 0 0" />
+          xyz="0.024842 -0.00021599 0.048722"
+          rpy="0 0 0" />
       <mass
-        value="0.08" />
+          value="0.08" />
       <inertia
-        ixx="8.4498E-05"
-        ixy="-1.8832E-09"
-        ixz="1.705E-07"
-        iyy="7.8484E-05"
-        iyz="-2.2039E-07"
-        izz="7.3534E-05" />
+          ixx="8.4498E-05"
+          ixy="-1.8832E-09"
+          ixz="1.705E-07"
+          iyy="7.8484E-05"
+          iyz="-2.2039E-07"
+          izz="7.3534E-05" />
     </inertial>
     <visual>
       <origin
-        xyz="0 0 0"
-        rpy="0 0 0" />
-      <geometry>
-        <mesh
-          filename="package://birl_gripper_description/meshes/female_camera/camera_frame.STL" />
+          xyz="0 0 0"
+          rpy="0 0 0" />
+      <geometry>
+        <mesh
+            filename="package://birl_gripper_description/meshes/male_camera/camera_frame.STL" />
       </geometry>
       <material
-        name="">
+          name="">
         <color
-          rgba="0.2 0.2 0.2 1" />
+            rgba="0.2 0.2 0.2 1" />
       </material>
     </visual>
     <collision>
       <origin
-        xyz="0 0 0"
-        rpy="0 0 0" />
-      <geometry>
-        <mesh
-          filename="package://birl_gripper_description/meshes/female_camera/camera_frame.STL" />
+          xyz="0 0 0"
+          rpy="0 0 0" />
+      <geometry>
+        <mesh
+            filename="package://birl_gripper_description/meshes/male_camera/camera_frame.STL" />
       </geometry>
     </collision>
   </link>
+  <joint name="${side}_gripper_base_camera_frame" type="fixed">
+    <origin rpy="0 0 ${pi}" xyz="0.020 0 0"/>
+    <parent link="${side}_hand"/>
+    <child link="${side}_camera_frame"/>
+  </joint>
+  <gazebo reference="${side}_camera_frame">
+    <mu1>1000</mu1>
+    <mu2>1000</mu2>
+    <fdir1>0.0 0.0 1.0</fdir1>
+    <kp>1e4</kp>
+    <kd>1.0</kd>
+    <material>Gazebo/Gold</material>
+    <self_collide>1</self_collide>
+  </gazebo>
+      <joint name="${side}_pa_endpoint" type="fixed">
+      <origin rpy="0 0 0" xyz="0 0 0.052"/>
+      <parent link="${side}_gripper_base"/>
+      <child link="${side}_pa_gripper"/>
+    </joint>
+    <!-- Electric Gripper Tip link -->
+    <link name="${side}_pa_gripper">
+      <inertial>
+        <origin rpy="0 0 0" xyz="0 0 0"/>
+        <mass value="0.0001"/>
+        <inertia ixx="0" ixy="0" ixz="0" iyy="0" iyz="0" izz="0.0"/>
+      </inertial>
+    </link>
+</xacro:if>
+<!--<xacro:if value="${male_holder}">-->
+<xacro:if value="${male_holder}">
   <link
-    name="${side}_female_holder">
+      name="${side}_male_holder">
     <inertial>
       <origin
-        xyz="1.2757E-10 9.385E-11 -0.001967"
-        rpy="0 0 0" />
+          xyz="1.2757E-10 9.385E-11 -0.001967"
+          rpy="0 0 0" />
       <mass
-        value="0.0301" />
+          value="0.0301" />
       <inertia
-        ixx="9.4008E-06"
-        ixy="-3.1962E-14"
-        ixz="3.1794E-15"
-        iyy="3.9813E-06"
-        iyz="2.3567E-15"
-        izz="1.3208E-05" />
+          ixx="9.4008E-06"
+          ixy="-3.1962E-14"
+          ixz="3.1794E-15"
+          iyy="3.9813E-06"
+          iyz="2.3567E-15"
+          izz="1.3208E-05" />
     </inertial>
     <visual>
       <origin
-        xyz="0 0 0"
-        rpy="0 0 0" />
-      <geometry>
-        <mesh
-          filename="package://birl_gripper_description/meshes/female_camera/female_holder.STL" />
+          xyz="0 0 0"
+          rpy="0 0 0" />
+      <geometry>
+        <mesh
+            filename="package://birl_gripper_description/meshes/male_camera/male_holder.STL" />
       </geometry>
       <material
-        name="">
+          name="">
         <color
-          rgba="0 0.552 0 1" />
+            rgba="0 0.552 0 1" />
       </material>
     </visual>
     <collision>
       <origin
-        xyz="0 0 0"
-        rpy="0 0 0" />
-      <geometry>
-        <mesh
-          filename="package://birl_gripper_description/meshes/female_camera/female_holder.STL" />
+          xyz="0 0 0"
+          rpy="0 0 0" />
+      <geometry>
+        <mesh
+            filename="package://birl_gripper_description/meshes/male_camera/male_holder.STL" />
       </geometry>
     </collision>
   </link>
   <joint
-    name="${side}_camera_frame_joint"
-    type="fixed">
+      name="${side}_camera_frame_joint"
+      type="fixed">
     <origin
-      xyz="0.025 -0.00031879 0.076"
-      rpy="4.7429E-14 8.4242E-30 1.4971E-16" />
+        xyz="0.025 -0.00031879 0.076"
+        rpy="4.7429E-14 8.4242E-30 1.4971E-16" />
     <parent
-      link="${side}_camera_frame" />
+        link="${side}_camera_frame" />
     <child
-      link="${side}_female_holder" />
+        link="${side}_male_holder" />
     <axis
-      xyz="0 0 0" />
+        xyz="0 0 0" />
   </joint>
-    <joint name="${side}_gripper_base_camera_frame" type="fixed">
-      <origin rpy="0 0 ${pi}" xyz="0.020 0 0"/>
-      <parent link="${side}_hand"/>
-      <child link="${side}_camera_frame"/>
-    </joint>
-        </xacro:if>
+  <gazebo reference="${side}_male_holder">
+    <mu1>1000</mu1>
+    <mu2>1000</mu2>
+    <fdir1>0.0 0.0 1.0</fdir1>
+    <kp>1e4</kp>
+    <kd>1.0</kd>
+    <material>Gazebo/Purple</material>
+    <self_collide>1</self_collide>
+  </gazebo>
+</xacro:if>
     <!-- Left finger link -->
     <xacro:property name="finger_length" value="0.0" scope="global"/>
