Commit message: change to right hand and rename files

File: birl_baxter_description/urdf/baxter_element/baxter_pa/baxter_pa_box.urdf.xacro (robot description, xacro)
@@ -10,4 +10,8 @@
   <xacro:arg name="left_male_holder" default="true"/>
   <xacro:arg name="right_male_holder" default="true"/>
+    <!--options:
+      finger = extended_wide extended_narrow standard_narrow standard_wide pa_finger
+      finger_slot = 1-6
+      fing_tip = basic_hard_tip basic_soft_tip half_round_tip paddle_tip none-->
   <xacro:arg name="l_finger"       default="pa_finger"/>
   <xacro:arg name="l_finger_slot"  default="6"/>
@@ -52,8 +56,8 @@
     <xacro:include filename="$(find birl_baxter_description)/urdf/box/box_male/robots/box_male.URDF" >
     </xacro:include>
-  <joint name="left_male_box_joint" type="fixed">
+  <joint name="right_male_box_joint" type="fixed">
       <origin rpy="0 0 0" xyz="0 0 0.015"/>
-      <parent link="left_male_holder" />
-      <child link="left_box_male"/>
+      <parent link="right_male_holder" />
+      <child link="box_male"/>
   </joint>
   <!-- Table -->
@@ -85,2 +89,19 @@
     </joint>
 </robot>
+<!--      <xacro:include filename="$(find birl_baxter_description)/urdf/snap/snap_female/robots/snap_female.URDF" >
+      </xacro:include>
+   <joint name="male_box_joint" type="fixed">
+      <origin rpy="0 0 0" xyz="0.6 0 -0.115"/>
+      <parent link="base" />
+      <child link="female_snap"/>
+  </joint>
+-->
+<!--
+    <xacro:include filename="$(find birl_baxter_description)/urdf/snap/snap_male/robots/snap_male.URDF" >
+    </xacro:include>
+   <joint name="left_male_snap_joint" type="fixed">
+      <origin rpy="${pi} 0 0" xyz="0 0 0.01"/>
+      <parent link="left_male_holder" />
+      <child link="snap_male"/>
+  </joint>
+    -->

File: birl_baxter_description/urdf/baxter_element/baxter_pa/baxter_pa_box2.urdf.xacro (robot description, xacro)
@@ -10,16 +10,16 @@
   <xacro:arg name="left_male_holder" default="false"/>
   <xacro:arg name="right_male_holder" default="false"/>
+  <!--options:
+      finger = extended_wide extended_narrow standard_narrow standard_wide pa_finger
+      finger_slot = 1-6
+      fing_tip = basic_hard_tip basic_soft_tip half_round_tip paddle_tip none-->
   <xacro:arg name="l_finger"       default="standard_narrow"/>
   <xacro:arg name="l_finger_slot"  default="4"/>
   <xacro:arg name="l_finger_tip"   default="paddle_tip"/>
   <xacro:arg name="l_finger_grasp" default="inner"/>
-  <xacro:arg name="r_finger"       default="pa_finger"/>
-  <xacro:arg name="r_finger_slot"  default="6"/>
-  <xacro:arg name="r_finger_tip"   default="pa_tip"/>
+  <xacro:arg name="r_finger"       default="standard_narrow"/>
+  <xacro:arg name="r_finger_slot"  default="4"/>
+  <xacro:arg name="r_finger_tip"   default="paddle_tip"/>
   <xacro:arg name="r_finger_grasp" default="inner"/>
-  <!--options:
-      finger = extended_wide extended_narrow standard_narrow standard_wide pa_finger
-      finger_slot = 1-6
-      fing_tip = basic_hard_tip basic_soft_tip half_round_tip paddle_tip none-->
   <xacro:arg name="left_ft_sensor" default="true"/>
   <xacro:arg name="right_ft_sensor" default="true"/>

File: birl_baxter_description/urdf/baxter_element/baxter_pa/baxter_pa_snap.urdf.xacro (robot description, xacro)
@@ -8,4 +8,10 @@
   <xacro:arg name="right_camera_frame" default="true"/>
   <xacro:arg name="left_camera_frame" default="true"/>
+  <xacro:arg name="left_male_holder" default="true"/>
+  <xacro:arg name="right_male_holder" default="true"/>
+  <!--options:
+      finger = extended_wide extended_narrow standard_narrow standard_wide pa_finger
+      finger_slot = 1-6
+      fing_tip = basic_hard_tip basic_soft_tip half_round_tip paddle_tip none-->
   <xacro:arg name="l_finger"       default="pa_finger"/>
   <xacro:arg name="l_finger_slot"  default="6"/>
@@ -16,5 +22,5 @@
   <xacro:arg name="r_finger_tip"   default="pa_tip"/>
   <xacro:arg name="r_finger_grasp" default="inner"/>
-  <xacro:arg name="left_ft_sensor" default="false"/>
+  <xacro:arg name="left_ft_sensor" default="true"/>
   <xacro:arg name="right_ft_sensor" default="true"/>
   <!-- Baxter Base URDF -->
@@ -33,4 +39,5 @@
     <xacro:include filename="$(find birl_baxter_description)/urdf/baxter_element/left_end_pa_effector.urdf.xacro" >
       <xacro:arg name="left_camera_frame" default="$(left_camera_frame)"/>
+      <xacro:arg name="left_male_gripper" default="$(left_male_gripper)"/>
       <xacro:arg name="l_finger" default="$(l_finger)"/>
       <xacro:arg name="l_finger_slot" default="$(l_finger_slot)"/>
@@ -41,4 +48,5 @@
     <xacro:include filename="$(find birl_baxter_description)/urdf/baxter_element/right_end_pa_effector.urdf.xacro" >
       <xacro:arg name="right_camera_frame" default="$(right_camera_frame)"/>
+      <xacro:arg name="right_male_gripper" default="$(right_male_gripper)"/>
       <xacro:arg name="r_finger" default="$(r_finger)"/>
       <xacro:arg name="r_finger_slot" default="$(r_finger_slot)"/>
@@ -48,8 +56,18 @@
     <xacro:include filename="$(find birl_baxter_description)/urdf/snap/snap_male/robots/snap_male.URDF" >
     </xacro:include>
+  <joint name="right_male_snap_joint" type="fixed">
+    <origin rpy="${pi} 0 0" xyz="0 0 0.01"/>
+    <parent link="right_male_holder" />
+    <child link="snap_male"/>
+  </joint>
   <!-- Table -->
   <xacro:if value="$(arg table)">
     <xacro:include filename="$(find birl_baxter_description)/urdf/table/table.xacro">
     </xacro:include>
+    <joint name="table_fixed" type="fixed">
+      <origin rpy="0 0 0" xyz="0.0 0.0 -0.93"/>
+      <parent link="base"/>
+      <child link="table"/>
+    </joint>
   </xacro:if>
   <!-- Asus Xtion -->
@@ -57,6 +75,16 @@
     <xacro:include filename="$(find birl_baxter_description)/urdf/asus_xtion/asus_xtion.xacro">
     </xacro:include>
+    <joint name="camera_base_fixed" type="fixed">
+      <origin rpy="0 0 0" xyz="1.0 0.0 -0.93"/>
+      <parent link="base"/>
+      <child link="camera_base"/>
+    </joint>
   </xacro:if>
-      <xacro:include filename="$(find birl_baxter_description)/urdf/snap/snap_female/robots/snap_female.URDF" >
-    </xacro:include>
+  <xacro:include filename="$(find birl_baxter_description)/urdf/snap/snap_female/robots/snap_female.URDF" >
+  </xacro:include>
+   <joint name="female_snap_joint" type="fixed">
+      <origin rpy="0 0 0" xyz="0.6 0 -0.115"/>
+      <parent link="base" />
+      <child link="female_snap"/>
+  </joint>
 </robot>

File: birl_baxter_description/urdf/box/box_male/robots/box_male.URDF (robot description, URDF)
Before this commit: robot left_box_male, 1 links, 0 joints
Links:
- removed link left_box_male
- added link box_male, mass 0.01526; collision mesh filename=package://birl_baxter_description/urdf/box/box_male/meshes/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; visual mesh filename=package://birl_baxter_description/urdf/box/box_male/meshes/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

File: birl_baxter_description/urdf/snap/snap_female/robots/snap_female.URDF (robot description, URDF)
Before this commit: robot snap_female, 1 links, 1 joints
Joints:
- removed joint male_box_joint

File: birl_baxter_description/urdf/snap/snap_male/robots/snap_male.URDF (robot description, URDF)
Before this commit: robot snap_male, 1 links, 1 joints
Joints:
- removed joint left_male_snap_joint
