Commit message: find solution and fixed the problem in ft "fixed joint problem" make every fix joint to revolute

File: birl_baxter_description/urdf/baxter_element/baxter_pa/test.urdf (robot description, URDF)
Before this commit: robot baxter, 44 links, 41 joints
Links:
- added link FT_Top_Plate_right, mass 0.053196; collision mesh filename=package://birl_baxter_description/urdf/ft/meshes/FT_Top_Pla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; visual mesh filename=package://birl_baxter_description/urdf/ft/meshes/FT_Top_Pla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
- added link FT_bottom_plate_right, mass 0.051726; collision mesh filename=package://birl_baxter_description/urdf/ft/meshes/FT_bottom_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; visual mesh filename=package://birl_baxter_description/urdf/ft/meshes/FT_bottom_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
- added link FT_right, mass 1.4264; collision mesh filename=package://birl_baxter_description/urdf/ft/meshes/FT.STL; visual mesh filename=package://birl_baxter_description/urdf/ft/meshes/FT.STL
- added link asus_xtion, mass 0.440171; collision mesh filename=package://birl_baxter_description/meshes/asus_xtion/asus_xt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; visual mesh filename=package://birl_baxter_description/meshes/asus_xtion/asus_xt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
- added link box_female, mass 0.01501; collision mesh filename=package://birl_baxter_description/urdf/box/box_female/meshe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; visual mesh filename=package://birl_baxter_description/urdf/box/box_female/meshe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
- added link box_male, mass 0.01526; collision mesh filename=package://birl_baxter_description/urdf/box/box_male/meshes/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; visual mesh filename=package://birl_baxter_description/urdf/box/box_male/meshes/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
- added link camera_base, mass 60.86397744; collision mesh filename=package://birl_baxter_description/meshes/asus_xtion/camera_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; visual mesh filename=package://birl_baxter_description/meshes/asus_xtion/camera_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
- added link install_link, mass 0.547767; collision mesh filename=package://birl_baxter_description/meshes/asus_xtion/install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; visual mesh filename=package://birl_baxter_description/meshes/asus_xtion/install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
- added link l_gripper_l_finger, mass 0.02; collision mesh filename=package://birl_gripper_description/meshes/electric_gripper/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; visual mesh filename=package://birl_gripper_description/meshes/electric_gripper/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
- added link l_gripper_l_finger_tip, mass 0.01; collision box size=0.02 0.002 0.015; visual box size=0.02 0.002 0.015
- added link l_gripper_r_finger, mass 0.02; collision mesh filename=package://birl_gripper_description/meshes/electric_gripper/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; visual mesh filename=package://birl_gripper_description/meshes/electric_gripper/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
- added link l_gripper_r_finger_tip, mass 0.01; collision box size=0.02 0.002 0.015; visual box size=0.02 0.002 0.015
- added link left_camera_frame, mass 0.08; collision mesh filename=package://birl_gripper_description/meshes/male_camera/camer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; visual mesh filename=package://birl_gripper_description/meshes/male_camera/camer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
- added link left_gripper, mass 0.0001
- added link left_gripper_base, mass 0.3; collision cylinder length=0.1 radius=0.029; visual mesh filename=package://birl_gripper_description/meshes/electric_gripper/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
- added link left_male_holder, mass 0.0301; collision mesh filename=package://birl_gripper_description/meshes/male_camera/male_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; visual mesh filename=package://birl_gripper_description/meshes/male_camera/male_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
- added link left_pa_gripper, mass 0.0001
- added link pedestal, mass 60.86397744; collision mesh filename=package://baxter_description/meshes/base/pedestal_link_coll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; visual mesh filename=package://baxter_description/meshes/base/PEDESTAL.DAE
- added link r_gripper_l_finger, mass 0.02; collision mesh filename=package://birl_gripper_description/meshes/electric_gripper/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; visual mesh filename=package://birl_gripper_description/meshes/electric_gripper/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
- added link r_gripper_l_finger_tip, mass 0.01; collision box size=0.02 0.002 0.015; visual box size=0.02 0.002 0.015
- added link r_gripper_r_finger, mass 0.02; collision mesh filename=package://birl_gripper_description/meshes/electric_gripper/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; visual mesh filename=package://birl_gripper_description/meshes/electric_gripper/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
- added link r_gripper_r_finger_tip, mass 0.01; collision box size=0.02 0.002 0.015; visual box size=0.02 0.002 0.015
- added link right_camera_frame, mass 0.08; collision mesh filename=package://birl_gripper_description/meshes/male_camera/camer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; visual mesh filename=package://birl_gripper_description/meshes/male_camera/camer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
- added link right_gripper, mass 0.0001
- added link right_gripper_base, mass 0.3; collision cylinder length=0.1 radius=0.029; visual mesh filename=package://birl_gripper_description/meshes/electric_gripper/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
- added link right_male_holder, mass 0.0301; collision mesh filename=package://birl_gripper_description/meshes/male_camera/male_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; visual mesh filename=package://birl_gripper_description/meshes/male_camera/male_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
- added link right_pa_gripper, mass 0.0001
- added link table, mass 60.86397744; collision mesh filename=package://birl_baxter_description/meshes/table/table.stl; visual mesh filename=package://birl_baxter_description/meshes/table/table.dae
Joints:
- added joint FT_Bottom_Joint_right: type fixed, parent FT_bottom_plate_right, child FT_right, origin xyz=0.041625 -0.00085087 0.040469 rpy=-3.1416 6.2028E-17 1.5708, axis 0 0 0
- added joint FT_Top_Joint_right: type revolute, parent FT_right, child FT_Top_Plate_right, origin xyz=0.00085087 -0.00087515 -0.0030305 rpy=3.1416 5.017E-16 1.5708, axis 0 0 1, limit lower=0 upper=0 effort=0.2 velocity=0.2
- added joint asus_xtion_fixed: type fixed, parent install_link, child asus_xtion, origin xyz=-0.0175 0 0.0 rpy=0 3.14159265359 1.57079632679
- added joint camera_base_fixed: type fixed, parent base, child camera_base, origin xyz=1.0 0.0 -0.93 rpy=0 0 0
- added joint female_box_joint: type fixed, parent base, child box_female, origin xyz=0.6 0 -0.115 rpy=0 0 0
- added joint install_link_fixed: type fixed, parent camera_base, child install_link, origin xyz=-0.35 -0.05 1.5 rpy=0 0 0
- added joint l_gripper_l_finger_joint: type prismatic, parent left_gripper_base, child l_gripper_l_finger, origin xyz=0.0 0.0365 0.02 rpy=0 0 0, axis 0 1 0, limit lower=0.0 upper=0.020833 effort=20.0 velocity=5.0
- added joint l_gripper_l_finger_tip_joint: type fixed, parent l_gripper_l_finger, child l_gripper_l_finger_tip, origin xyz=0 0 0 rpy=0 0 0
- added joint l_gripper_r_finger_joint: type prismatic, parent left_gripper_base, child l_gripper_r_finger, origin xyz=0.0 -0.0365 0.02 rpy=0 0 0, axis 0 1 0, limit lower=-0.020833 upper=0.0 effort=20.0 velocity=5.0, mimic joint=l_gripper_l_finger_joint multiplier=-1.0
- added joint l_gripper_r_finger_tip_joint: type fixed, parent l_gripper_r_finger, child l_gripper_r_finger_tip, origin xyz=0 0 0 rpy=0 0 0
- added joint left_camera_frame_joint: type fixed, parent left_camera_frame, child left_male_holder, origin xyz=0.025 -0.00031879 0.076 rpy=4.7429E-14 8.4242E-30 1.4971E-16, axis 0 0 0
- added joint left_endpoint: type fixed, parent left_gripper_base, child left_gripper, origin xyz=0 0 0.1327 rpy=0 0 0
- added joint left_gripper_base: type fixed, parent left_hand, child left_gripper_base, origin xyz=0 0 0.025 rpy=0 0 0
- added joint left_gripper_base_camera_frame: type fixed, parent left_hand, child left_camera_frame, origin xyz=0.020 0 0 rpy=0 0 3.14159265359
- added joint left_hand: type fixed, parent left_wrist, child left_hand, origin xyz=0 0 0.11355 rpy=0 0 0, axis 0 0 1
- added joint left_pa_endpoint: type fixed, parent left_gripper_base, child left_pa_gripper, origin xyz=0 0 0.052 rpy=0 0 0
- added joint pedestal_fixed: type fixed, parent torso, child pedestal, origin xyz=0.0 0.0 0.0 rpy=0 0 0
- added joint r_gripper_l_finger_joint: type prismatic, parent right_gripper_base, child r_gripper_l_finger, origin xyz=0.0 0.0365 0.02 rpy=0 0 0, axis 0 1 0, limit lower=0.0 upper=0.020833 effort=20.0 velocity=5.0
- added joint r_gripper_l_finger_tip_joint: type fixed, parent r_gripper_l_finger, child r_gripper_l_finger_tip, origin xyz=0 0 0 rpy=0 0 0
- added joint r_gripper_r_finger_joint: type prismatic, parent right_gripper_base, child r_gripper_r_finger, origin xyz=0.0 -0.0365 0.02 rpy=0 0 0, axis 0 1 0, limit lower=-0.020833 upper=0.0 effort=20.0 velocity=5.0, mimic joint=r_gripper_l_finger_joint multiplier=-1.0
- added joint r_gripper_r_finger_tip_joint: type fixed, parent r_gripper_r_finger, child r_gripper_r_finger_tip, origin xyz=0 0 0 rpy=0 0 0
- added joint right_camera_frame_joint: type fixed, parent right_camera_frame, child right_male_holder, origin xyz=0.025 -0.00031879 0.076 rpy=4.7429E-14 8.4242E-30 1.4971E-16, axis 0 0 0
- added joint right_endpoint: type fixed, parent right_gripper_base, child right_gripper, origin xyz=0 0 0.1327 rpy=0 0 0
- added joint right_ft_hand: type fixed, parent right_wrist, child FT_bottom_plate_right, origin xyz=0.025 0 0.11355 rpy=3.14159265359 3.14159265359 0
- added joint right_gripper_base: type fixed, parent right_hand, child right_gripper_base, origin xyz=0 0 0.025 rpy=0 0 0
- added joint right_gripper_base_camera_frame: type fixed, parent right_hand, child right_camera_frame, origin xyz=0.020 0 0 rpy=0 0 3.14159265359
- added joint right_hand: type fixed, parent right_wrist, child right_hand, origin xyz=0 0 0.169 rpy=0 0 0, axis 0 0 1
- added joint right_male_box_joint: type fixed, parent right_male_holder, child box_male, origin xyz=0 0 0.015 rpy=0 0 0
- added joint right_pa_endpoint: type fixed, parent right_gripper_base, child right_pa_gripper, origin xyz=0 0 0.052 rpy=0 0 0
- added joint table_fixed: type fixed, parent base, child table, origin xyz=0.0 0.0 -0.93 rpy=0 0 0

File: birl_baxter_description/urdf/ft/robots/FT_Electric_left.URDF (robot description, URDF)
Before this commit: robot FT_Electric_left, 3 links, 2 joints
Joints:
- joint FT_Top_Joint_left: limit lower=0 upper=0.0006 effort=0.001 velocity=0.001 -> lower=0 upper=0 effort=0.2 velocity=0.2; type fixed -> revolute

File: birl_baxter_description/urdf/ft/robots/FT_Electric_right.URDF (robot description, URDF)
Before this commit: robot FT_Electric_right, 3 links, 2 joints
Joints:
- joint FT_Top_Joint_right: limit lower=0 upper=0.0006 effort=0.001 velocity=0.001 -> lower=0 upper=0 effort=0.2 velocity=0.2; type fixed -> revolute
