Commit message: modify baxter_ft.urdf.xacro

File: birl_baxter_description/urdf/baxter_element/baxter/baxter_ft.urdf (robot description, URDF)
Before this commit: robot baxter, 64 links, 63 joints
Links:
- removed link table
- link l_gripper_l_finger: geometry collision box size=0.01 0.0135 0.1127; collision box size=0.01 0.05 0.017
- link l_gripper_l_finger_tip: geometry collision box size=0.042 0.0065 0.037; visual mesh filename=package://rethink_ee_description/meshes/electric_gripper/fi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
- link l_gripper_r_finger: geometry collision box size=0.01 0.0135 0.1127; collision box size=0.01 0.05 0.017
- link l_gripper_r_finger_tip: geometry collision box size=0.042 0.0065 0.037; visual mesh filename=package://rethink_ee_description/meshes/electric_gripper/fi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
- link left_gripper_base: geometry collision cylinder length=0.1 radius=0.029; visual mesh filename=package://rethink_ee_description/meshes/electric_gripper/el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
- link r_gripper_l_finger: geometry collision box size=0.01 0.0135 0.1127; collision box size=0.01 0.05 0.017
- link r_gripper_l_finger_tip: geometry collision box size=0.042 0.0065 0.037; visual mesh filename=package://rethink_ee_description/meshes/electric_gripper/fi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
- link r_gripper_r_finger: geometry collision box size=0.01 0.0135 0.1127; collision box size=0.01 0.05 0.017
- link r_gripper_r_finger_tip: geometry collision box size=0.042 0.0065 0.037; visual mesh filename=package://rethink_ee_description/meshes/electric_gripper/fi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
- link right_gripper_base: geometry collision cylinder length=0.1 radius=0.029; visual mesh filename=package://rethink_ee_description/meshes/electric_gripper/el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
Joints:
- removed joint l_ft_bottom_hand
- removed joint r_ft_bottom_hand
- removed joint table_fixed
- added joint left_ft_hand: type fixed, parent left_wrist, child FT_bottom_plate_left, origin xyz=0.025 0 0.11355 rpy=3.14159265359 3.14159265359 0
- added joint right_ft_hand: type fixed, parent right_wrist, child FT_bottom_plate_right, origin xyz=0.025 0 0.11355 rpy=3.14159265359 3.14159265359 0
- joint l_gripper_l_finger_tip_joint: origin xyz=0.0 0.01725 0.075 rpy=0 0 0 -> xyz=0.0 0.01725 0.1127 rpy=0 0 0
- joint l_gripper_r_finger_tip_joint: origin xyz=0.0 -0.01725 0.075 rpy=0 0 0 -> xyz=0.0 -0.01725 0.1127 rpy=0 0 0
- joint left_endpoint: origin xyz=0 0 0.095 rpy=0 0 0 -> xyz=0 0 0.1327 rpy=0 0 0
- joint left_gripper_base: parent FT_Top_Plate_left -> left_hand
- joint left_hand: origin xyz=0 0 0.11355 rpy=0 0 0 -> xyz=0 0 0.169 rpy=0 0 0
- joint r_gripper_l_finger_tip_joint: origin xyz=0.0 0.05503 0.1127 rpy=0 0 0 -> xyz=0.0 0.01725 0.1127 rpy=0 0 0
- joint r_gripper_r_finger_tip_joint: origin xyz=0.0 -0.05503 0.1127 rpy=0 0 0 -> xyz=0.0 -0.01725 0.1127 rpy=0 0 0
- joint right_gripper_base: parent FT_Top_Plate_right -> right_hand
- joint right_hand: origin xyz=0 0 0.11355 rpy=0 0 0 -> xyz=0 0 0.169 rpy=0 0 0

File: birl_baxter_description/urdf/baxter_element/baxter_base/baxter_base_ft.urdf.xacro (robot description, xacro)
@@ -589,5 +589,4 @@
     <dynamics damping="0.7" friction="0.0"/>
   </joint>
-  <!--
   <joint name="right_hand" type="fixed">
     <origin rpy="0 0 0" xyz="0 0 0.11355"/>
@@ -596,5 +595,4 @@
     <child link="right_hand"/>
     </joint>
-    -->
   <joint name="right_hand_camera" type="fixed">
     <origin rpy="0 0 -1.57079633" xyz="0.03825 0.012 0.015355"/>
@@ -959,5 +957,4 @@
     <dynamics damping="0.7" friction="0.0"/>
   </joint>
-  <!--
   <joint name="left_hand" type="fixed">
     <origin rpy="0 0 0" xyz="0 0 0.11355"/>
@@ -966,5 +963,4 @@
     <child link="left_hand"/>
     </joint>
-    -->
   <joint name="left_hand_camera" type="fixed">
     <origin rpy="0 0 -1.57079633" xyz="0.03825 0.012 0.015355"/>
@@ -989,14 +985,9 @@
   <xacro:if value="$(arg right_ft_sensor)">
     <!-- change compared to baxter_base.urdf.xacro -->
-    <joint name="right_hand" type="fixed">
-      <origin rpy="0 0 0" xyz="0 0 0.169"/>
-      <axis xyz="0 0 1"/>
-      <parent link="right_wrist"/>
-      <child link="right_hand"/>
-    </joint>
-    <xacro:include filename="$(find birl_baxter_description)/urdf/ft/robots/FT_Electric_right.URDF"/>
-    <joint name="right_ft_hand" type="fixed">
-      <origin rpy="${pi} ${pi} 0" xyz="0.025 0 0.11355"/>
-      <parent link="right_wrist"/>
+    <xacro:include filename="$(find birl_baxter_description)/urdf/ft/robots/FT_Electric_right.URDF">
+    </xacro:include>
+    <joint name="r_ft_bottom_hand" type="fixed">
+      <origin rpy="${pi} ${pi} 0" xyz="0.02 0 0"/>
+      <parent link="right_hand"/>
       <child link="FT_bottom_plate_right"/>
     </joint>
@@ -1011,26 +1002,14 @@
       </plugin>
     </gazebo>
+<!--ft sensor library link-->
   </xacro:if>
-  <xacro:unless value="$(arg right_ft_sensor)">
-    <joint name="right_hand" type="fixed">
-      <origin rpy="0 0 0" xyz="0 0 0.11355"/>
-      <axis xyz="0 0 1"/>
-      <parent link="right_wrist"/>
-      <child link="right_hand"/>
-    </joint>
-  </xacro:unless>
-   <xacro:if value="$(arg left_ft_sensor)">
-    <!-- change compared to baxter_base.urdf.xacro -->
-    <joint name="left_hand" type="fixed">
-      <origin rpy="0 0 0" xyz="0 0 0.169"/>
-      <axis xyz="0 0 1"/>
-      <parent link="left_wrist"/>
-      <child link="left_hand"/>
-    </joint>
-    <xacro:include filename="$(find birl_baxter_description)/urdf/ft/robots/FT_Electric_left.URDF"/>
-    <joint name="left_ft_hand" type="fixed">
-      <origin rpy="${pi} ${pi} 0" xyz="0.025 0 0.11355"/>
-      <parent link="left_wrist"/>
-      <child link="FT_bottom_plate_left"/>
+<!--# end xacro if -->
+  <xacro:if value="$(arg left_ft_sensor)">
+    <xacro:include filename="$(find birl_baxter_description)/urdf/ft/robots/FT_Electric_left.URDF">
+    </xacro:include>
+    <joint name="l_ft_bottom_hand" type="fixed">
+        <origin rpy="${pi} ${pi} 0" xyz="0.02 0 0"/>
+        <parent link="left_hand"/>
+        <child link="FT_bottom_plate_left"/>
     </joint>
     <gazebo reference="FT_Top_Joint_left">
@@ -1045,11 +1024,3 @@
     </gazebo>
   </xacro:if>
-  <xacro:unless value="$(arg left_ft_sensor)">
-    <joint name="left_hand" type="fixed">
-      <origin rpy="0 0 0" xyz="0 0 0.11355"/>
-      <axis xyz="0 0 1"/>
-      <parent link="left_wrist"/>
-      <child link="left_hand"/>
-    </joint>
-  </xacro:unless>
 </robot>

File: birl_baxter_description/urdf/baxter_element/baxter_ft/baxter_ft.urdf.xacro (robot description, xacro)
@@ -4,5 +4,5 @@
   <xacro:arg name="pedestal" default="true"/>
   <!-- TODO: have an arg for pa_demo that sets correct eef's/table/xtion -->
-  <xacro:arg name="table" default="false"/>
+  <xacro:arg name="table" default="true"/>
   <xacro:arg name="asus_xtion" default="false"/>
   <xacro:arg name="right_camera_frame" default="false"/>

File: birl_gripper_description/urdf/electric_gripper/rethink_electric_pa_gripper.xacro (robot description, xacro)
@@ -202,5 +202,5 @@
     <joint name="${side}_gripper_base" type="fixed">
       <origin rpy="0 0 0" xyz="0 0 0.025"/>
-      <parent link="${side}_hand"/>
+      <parent link="FT_Top_Plate_${side}"/>
       <child link="${side}_gripper_base"/>
     </joint>
